Commit message: zeroRPC bridge added.

File: rob2004/assets/robot/urdf/pupper_v3.urdf (robot description, URDF)
Before this commit: robot pupper_v3, 13 links, 12 joints
Links:
- link base_link: geometry collision box size=0.09014 0.12758 0.25943; visual mesh filename=../meshes/stl/BodyV4v70_001.stl scale=1.00000 1.00000 1.00000
- link leg_back_l_1: geometry visual mesh filename=../meshes/stl/LegAssemblyForFlangedv26_013.stl scale=-1.00000 -1.00000 -1.00000
- link leg_back_l_2: geometry collision cylinder length=0.03000 radius=0.02500; visual mesh filename=../meshes/stl/LegAssemblyForFlangedv26_014.stl scale=-1.00000 -1.00000 -1.00000
- link leg_back_l_3: geometry collision sphere radius=0.01995; visual mesh filename=../meshes/stl/LegAssemblyForFlangedv26_015.stl scale=-1.00000 -1.00000 -1.00000
- link leg_back_r_1: geometry visual mesh filename=../meshes/stl/LegAssemblyForFlangedv26_005.stl scale=1.00000 1.00000 1.00000
- link leg_back_r_2: geometry collision cylinder length=0.03000 radius=0.02500; visual mesh filename=../meshes/stl/LegAssemblyForFlangedv26_006.stl scale=1.00000 1.00000 1.00000
- link leg_back_r_3: geometry collision sphere radius=0.01995; visual mesh filename=../meshes/stl/LegAssemblyForFlangedv26_007.stl scale=1.00000 1.00000 1.00000
- link leg_front_l_1: geometry visual mesh filename=../meshes/stl/LegAssemblyForFlangedv26_010.stl scale=-1.00000 -1.00000 -1.00000
- link leg_front_l_2: geometry collision cylinder length=0.03000 radius=0.02500; visual mesh filename=../meshes/stl/LegAssemblyForFlangedv26_011.stl scale=-1.00000 -1.00000 -1.00000
- link leg_front_l_3: geometry collision sphere radius=0.01995; visual mesh filename=../meshes/stl/LegAssemblyForFlangedv26_012.stl scale=-1.00000 -1.00000 -1.00000
- link leg_front_r_1: geometry visual mesh filename=../meshes/stl/LegAssemblyForFlangedv26_001.stl scale=1.00000 1.00000 1.00000
- link leg_front_r_2: geometry collision cylinder length=0.03000 radius=0.02500; visual mesh filename=../meshes/stl/LegAssemblyForFlangedv26_002.stl scale=1.00000 1.00000 1.00000
- link leg_front_r_3: geometry collision sphere radius=0.01995; visual mesh filename=../meshes/stl/LegAssemblyForFlangedv26_003.stl scale=1.00000 1.00000 1.00000
